File: Hardware/0.3/usb-hub.sch (KiCad schematic (older format))
At the start: 27 parts, among them J3 USB_C_Receptacle_USB2.0, J4 USB_C_Receptacle_USB2.0, J5 USB_C_Receptacle_USB2.0, U1 TPD2S017, U3 CY7C65632-28LTXCT, Y2 12MHz

Commit message: changing sw15/16 code
Parts:
- C12, C14, C15, C16, C21: Digikey PN (none) -> 1276-1000-1-ND; MPN (none) -> CL10B104KB8NNNC; Substitue Allowed? (none) -> Y
- C13: Digikey PN (none) -> 1276-1871-1-ND; MPN (none) -> CL10A106MP8NNNC; Substitue Allowed? (none) -> Y
- C17, C18: Digikey PN (none) -> 1276-2228-1-ND; MPN (none) -> CL10C220JB8NFNC; Substitue Allowed? (none) -> Y
- C19, C20, C22: Digikey PN (none) -> 1276-1866-1-ND; MPN (none) -> CL10A105MP8NNNC; Substitue Allowed? (none) -> Y
- FB1, FB2, FB3, FB4: Digikey PN (none) -> 490-1014-1-ND; Substitue Allowed? (none) -> Y
- J3, J4, J5: Notes (none) -> Cannot source from Digikey, available on AliExpress: https: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; Substitue Allowed? (none) -> N
- R10, R13, R9: Digikey PN (none) -> CR0603-JW-104ELFCT-ND; MPN (none) -> CR0603-JW-104ELF; Substitue Allowed? (none) -> Y
- R12: Digikey PN (none) -> CR0603-JW-103ELFCT-ND; MPN (none) -> CR0603-JW-103ELF; Substitue Allowed? (none) -> Y
- R14: Digikey PN (none) -> RHM649CFCT-ND; MPN (none) -> MCR03ERTF6490; Notes (none) -> Cannot source from LCSC, no substitutes available; Substitue Allowed? (none) -> Y
- RN5: Digikey PN (none) -> RAVF104DJT10K0CT-ND; MPN (none) -> RAVF104DJT10K0; Substitue Allowed? (none) -> Y
- U1: Notes (none) -> Cannot source from LCSC, no substitutes available; Substitue Allowed? (none) -> N
- U3: Digikey PN (none) -> 428-3156-1-ND; Substitue Allowed? (none) -> N
- Y2: Digikey PN (none) -> 535-9826-1-ND; Substitue Allowed? (none) -> Y
Changed lines of the file:
@@
 F 4 "CY7C65632-28LTXCT" H 5000 1575 50  0001 C CNN "MPN"
 F 5 "C466886" H 5000 1575 50  0001 C CNN "LCSC PN"
+F 6 "428-3156-1-ND" H 5000 1575 50  0001 C CNN "Digikey PN"
+F 7 "N" H 5000 1575 50  0001 C CNN "Substitue Allowed?"
 	1    5000 1575
 	1    0    0    -1
@@
 F 4 "C19330" H 1600 6750 50  0001 C CNN "LCSC PN"
 F 5 "BLM18AG601SN1D" H 1600 6750 50  0001 C CNN "MPN"
+F 6 "490-1014-1-ND" H 1600 6750 50  0001 C CNN "Digikey PN"
+F 7 "Y" H 1600 6750 50  0001 C CNN "Substitue Allowed?"
 	1    1600 6750
 	-1   0    0    1
@@
 F 2 "Capacitor_SMD:C_0603_1608Metric" H 1338 6900 50  0001 C CNN
 F 3 "~" H 1300 7050 50  0001 C CNN
+F 4 "1276-1000-1-ND" H 1300 7050 50  0001 C CNN "Digikey PN"
+F 5 "CL10B104KB8NNNC" H 1300 7050 50  0001 C CNN "MPN"
+F 6 "Y" H 1300 7050 50  0001 C CNN "Substitue Allowed?"
 	1    1300 7050
 	1    0    0    -1
@@
 F 2 "Capacitor_SMD:C_0603_1608Metric" H 1888 6900 50  0001 C CNN
 F 3 "~" H 1850 7050 50  0001 C CNN
+F 4 "1276-1871-1-ND " H 1850 7050 50  0001 C CNN "Digikey PN"
+F 5 "CL10A106MP8NNNC " H 1850 7050 50  0001 C CNN "MPN"
+F 6 "Y" H 1850 7050 50  0001 C CNN "Substitue Allowed?"
 	1    1850 7050
 	1    0    0    -1
@@
 F 2 "Capacitor_SMD:C_0603_1608Metric" H 2363 6775 50  0001 C CNN
 F 3 "~" H 2325 6925 50  0001 C CNN
+F 4 "1276-1000-1-ND" H 2325 6925 50  0001 C CNN "Digikey PN"
+F 5 "CL10B104KB8NNNC" H 2325 6925 50  0001 C CNN "MPN"
+F 6 "Y" H 2325 6925 50  0001 C CNN "Substitue Allowed?"
 	1    2325 6925
 	1    0    0    -1
@@
 F 2 "Capacitor_SMD:C_0603_1608Metric" H 2788 6775 50  0001 C CNN
 F 3 "~" H 2750 6925 50  0001 C CNN
+F 4 "1276-1000-1-ND" H 2750 6925 50  0001 C CNN "Digikey PN"
+F 5 "CL10B104KB8NNNC" H 2750 6925 50  0001 C CNN "MPN"
+F 6 "Y" H 2750 6925 50  0001 C CNN "Substitue Allowed?"
 	1    2750 6925
 	1    0    0    -1
@@
 F 2 "Capacitor_SMD:C_0603_1608Metric" H 3213 6775 50  0001 C CNN
 F 3 "~" H 3175 6925 50  0001 C CNN
+F 4 "1276-1000-1-ND" H 3175 6925 50  0001 C CNN "Digikey PN"
+F 5 "CL10B104KB8NNNC" H 3175 6925 50  0001 C CNN "MPN"
+F 6 "Y" H 3175 6925 50  0001 C CNN "Substitue Allowed?"
 	1    3175 6925
 	1    0    0    -1
@@
 F 2 "Capacitor_SMD:C_0603_1608Metric" H 3638 6775 50  0001 C CNN
 F 3 "~" H 3600 6925 50  0001 C CNN
+F 4 "1276-1866-1-ND " H 3600 6925 50  0001 C CNN "Digikey PN"
+F 5 "CL10A105MP8NNNC " H 3600 6925 50  0001 C CNN "MPN"
+F 6 "Y" H 3600 6925 50  0001 C CNN "Substitue Allowed?"
 	1    3600 6925
 	1    0    0    -1
@@
 F 2 "Capacitor_SMD:C_0603_1608Metric" H 4013 6775 50  0001 C CNN
 F 3 "~" H 3975 6925 50  0001 C CNN
+F 4 "1276-1866-1-ND " H 3975 6925 50  0001 C CNN "Digikey PN"
+F 5 "CL10A105MP8NNNC " H 3975 6925 50  0001 C CNN "MPN"
+F 6 "Y" H 3975 6925 50  0001 C CNN "Substitue Allowed?"
 	1    3975 6925
 	1    0    0    -1
@@
 F 2 "Capacitor_SMD:C_0603_1608Metric" H 4413 6775 50  0001 C CNN
 F 3 "~" H 4375 6925 50  0001 C CNN
+F 4 "1276-1000-1-ND" H 4375 6925 50  0001 C CNN "Digikey PN"
+F 5 "CL10B104KB8NNNC" H 4375 6925 50  0001 C CNN "MPN"
+F 6 "Y" H 4375 6925 50  0001 C CNN "Substitue Allowed?"
 	1    4375 6925
 	1    0    0    -1
@@
 F 2 "Capacitor_SMD:C_0603_1608Metric" H 4863 6775 50  0001 C CNN
 F 3 "~" H 4825 6925 50  0001 C CNN
+F 4 "1276-1866-1-ND " H 4825 6925 50  0001 C CNN "Digikey PN"
+F 5 "CL10A105MP8NNNC " H 4825 6925 50  0001 C CNN "MPN"
+F 6 "Y" H 4825 6925 50  0001 C CNN "Substitue Allowed?"
 	1    4825 6925
 	1    0    0    -1
@@
 F 2 "Resistor_SMD:R_0603_1608Metric" V 4605 3125 50  0001 C CNN
 F 3 "~" H 4675 3125 50  0001 C CNN
+F 4 "CR0603-JW-103ELFCT-ND  " H 4675 3125 50  0001 C CNN "Digikey PN"
+F 5 "CR0603-JW-103ELF " H 4675 3125 50  0001 C CNN "MPN"
+F 6 "Y" H 4675 3125 50  0001 C CNN "Substitue Allowed?"
 	1    4675 3125
 	0    1    1    0
@@
 F 2 "Capacitor_SMD:C_0603_1608Metric" H 3313 2725 50  0001 C CNN
 F 3 "~" H 3275 2875 50  0001 C CNN
+F 4 "1276-2228-1-ND  " H 3275 2875 50  0001 C CNN "Digikey PN"
+F 5 "CL10C220JB8NFNC " H 3275 2875 50  0001 C CNN "MPN"
+F 6 "Y" H 3275 2875 50  0001 C CNN "Substitue Allowed?"
 	1    3275 2875
 	0    1    1    0
@@
 F 2 "Capacitor_SMD:C_0603_1608Metric" H 3313 2325 50  0001 C CNN
 F 3 "~" H 3275 2475 50  0001 C CNN
+F 4 "1276-2228-1-ND  " H 3275 2475 50  0001 C CNN "Digikey PN"
+F 5 "CL10C220JB8NFNC " H 3275 2475 50  0001 C CNN "MPN"
+F 6 "Y" H 3275 2475 50  0001 C CNN "Substitue Allowed?"
 	1    3275 2475
 	0    1    1    0
@@
 F 4 "C276421" H 3675 2675 50  0001 C CNN "LCSC PN"
 F 5 "ABM8-12.000MHZ-B2-T" H 3675 2675 50  0001 C CNN "MPN"
+F 6 "535-9826-1-ND" H 3675 2675 50  0001 C CNN "Digikey PN"
+F 7 "Y" H 3675 2675 50  0001 C CNN "Substitue Allowed?"
 	1    3675 2675
 	0    1    1    0
@@
 F 2 "Resistor_SMD:R_0603_1608Metric" V 4605 3225 50  0001 C CNN
 F 3 "~" H 4675 3225 50  0001 C CNN
+F 4 "CR0603-JW-104ELFCT-ND " H 4675 3225 50  0001 C CNN "Digikey PN"
+F 5 "CR0603-JW-104ELF " H 4675 3225 50  0001 C CNN "MPN"
+F 6 "Y" H 4675 3225 50  0001 C CNN "Substitue Allowed?"
 	1    4675 3225
 	0    1    1    0
@@
 F 2 "Resistor_SMD:R_0603_1608Metric" V 4680 3625 50  0001 C CNN
 F 3 "~" H 4750 3625 50  0001 C CNN
+F 4 "RHM649CFCT-ND  " H 4750 3625 50  0001 C CNN "Digikey PN"
+F 5 "MCR03ERTF6490 " H 4750 3625 50  0001 C CNN "MPN"
+F 6 "Cannot source from LCSC, no substitutes available " H 4750 3625 50  0001 C CNN "Notes"
+F 7 "Y" H 4750 3625 50  0001 C CNN "Substitue Allowed?"
 	1    4750 3625
 	1    0    0    -1
@@
 F 3 "~" H 3725 3400 50  0001 C CNN
 F 4 "DNP" H 3850 3325 50  0000 C CNN "DNP"
+F 5 "CR0603-JW-104ELFCT-ND " H 3725 3400 50  0001 C CNN "Digikey PN"
+F 6 "CR0603-JW-104ELF " H 3725 3400 50  0001 C CNN "MPN"
+F 7 "Y" H 3725 3400 50  0001 C CNN "Substitue Allowed?"
 	1    3725 3400
 	1    0    0    -1
@@
 F 3 "~" H 3725 3750 50  0001 C CNN
 F 4 "" H 3850 3675 50  0000 C CNN "DNP"
+F 5 "CR0603-JW-104ELFCT-ND " H 3725 3750 50  0001 C CNN "Digikey PN"
+F 6 "CR0603-JW-104ELF " H 3725 3750 50  0001 C CNN "MPN"
+F 7 "Y" H 3725 3750 50  0001 C CNN "Substitue Allowed?"
 	1    3725 3750
 	1    0    0    -1
@@
 F 2 "Resistor_SMD:R_Array_Convex_4x0402" V 6350 7050 50  0001 C CNN
 F 3 "~" H 6075 7050 50  0001 C CNN
+F 4 "RAVF104DJT10K0CT-ND" H 6075 7050 50  0001 C CNN "Digikey PN"
+F 5 "RAVF104DJT10K0" H 6075 7050 50  0001 C CNN "MPN"
+F 6 "Y" H 6075 7050 50  0001 C CNN "Substitue Allowed?"
 	1    6075 7050
 	0    1    1    0
@@
 F 4 "C319148" H 10275 2375 50  0001 C CNN "LCSC PN"
 F 5 "U262-161N-4BVC11" H 10275 2375 50  0001 C CNN "MPN"
+F 6 "Cannot source from Digikey, available on AliExpress: https://www.aliexpress.com/item/33045191307.html" H 10275 2375 50  0001 C CNN "Notes"
+F 7 "N" H 10275 2375 50  0001 C CNN "Substitue Allowed?"
 	1    10275 2375
 	-1   0    0    -1
@@
 F 4 "C319148" H 8175 2350 50  0001 C CNN "LCSC PN"
 F 5 "U262-161N-4BVC11" H 8175 2350 50  0001 C CNN "MPN"
+F 6 "Cannot source from Digikey, available on AliExpress: https://www.aliexpress.com/item/33045191307.html" H 8175 2350 50  0001 C CNN "Notes"
+F 7 "N" H 8175 2350 50  0001 C CNN "Substitue Allowed?"
 	1    8175 2350
 	-1   0    0    -1
@@
 F 4 "C319148" H 10325 4575 50  0001 C CNN "LCSC PN"
 F 5 "U262-161N-4BVC11" H 10325 4575 50  0001 C CNN "MPN"
+F 6 "Cannot source from Digikey, available on AliExpress: https://www.aliexpress.com/item/33045191307.html" H 10325 4575 50  0001 C CNN "Notes"
+F 7 "N" H 10325 4575 50  0001 C CNN "Substitue Allowed?"
 	1    10325 4575
 	-1   0    0    -1
@@
 F 4 "C19330" H 9375 3975 50  0001 C CNN "LCSC PN"
 F 5 "BLM18AG601SN1D" H 9375 3975 50  0001 C CNN "MPN"
+F 6 "490-1014-1-ND" H 9375 3975 50  0001 C CNN "Digikey PN"
+F 7 "Y" H 9375 3975 50  0001 C CNN "Substitue Allowed?"
 	1    9375 3975
 	-1   0    0    1
@@
 F 4 "C19330" H 7325 1750 50  0001 C CNN "LCSC PN"
 F 5 "BLM18AG601SN1D" H 7325 1750 50  0001 C CNN "MPN"
+F 6 "490-1014-1-ND" H 7325 1750 50  0001 C CNN "Digikey PN"
+F 7 "Y" H 7325 1750 50  0001 C CNN "Substitue Allowed?"
 	1    7325 1750
 	-1   0    0    1
@@
 F 4 "C19330" H 9425 1775 50  0001 C CNN "LCSC PN"
 F 5 "BLM18AG601SN1D" H 9425 1775 50  0001 C CNN "MPN"
+F 6 "490-1014-1-ND" H 9425 1775 50  0001 C CNN "Digikey PN"
+F 7 "Y" H 9425 1775 50  0001 C CNN "Substitue Allowed?"
 	1    9425 1775
 	-1   0    0    1
@@
 F 4 "296-25216-1-ND " H 2075 2150 50  0001 C CNN "Digikey PN"
 F 5 "TPD2S017DBVR" H 2075 2150 50  0001 C CNN "MPN"
+F 6 "Cannot source from LCSC, no substitutes available " H 2075 2150 50  0001 C CNN "Notes"
+F 7 "N" H 2075 2150 50  0001 C CNN "Substitue Allowed?"
 	1    2075 2150
 	1    0    0    -1
