File: Hardware/0.3/Hub16.kicad_pcb (KiCad board)
At the start: 2 copper layers, 89 x 100 mm, 118 parts, among them J1 USB_C_Receptacle_USB2.0, J2 AVR-ISP-6, J3 USB_C_Receptacle_USB2.0, J4 USB_C_Receptacle_USB2.0, J5 USB_C_Receptacle_USB2.0, K1 KEYSW, K11 KEYSW, K12 KEYSW, K13 KEYSW, K14 KEYSW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

Commit message: update pnp tool
Parts:
- removed G***: LOGO, josh-logos:OSHW_Logo_3.6x3.6_F.Mask
- removed G***: LOGO, josh-logos:josh-johnson-logo-17x3
Connections:
- D32 pad 2: Net-(D32-Pad2) -> (no net)
- J1 pad A8: Net-(J1-PadA8) -> (no net)
- J1 pad B8: Net-(J1-PadB8) -> (no net)
- J3 pad A5: Net-(J3-PadA5) -> (no net)
- J3 pad A8: Net-(J3-PadA8) -> (no net)
- J3 pad B5: Net-(J3-PadB5) -> (no net)
- J3 pad B8: Net-(J3-PadB8) -> (no net)
- J4 pad A5: Net-(J4-PadA5) -> (no net)
- J4 pad A8: Net-(J4-PadA8) -> (no net)
- J4 pad B5: Net-(J4-PadB5) -> (no net)
- J4 pad B8: Net-(J4-PadB8) -> (no net)
- J5 pad A5: Net-(J5-PadA5) -> (no net)
- J5 pad A8: Net-(J5-PadA8) -> (no net)
- J5 pad B5: Net-(J5-PadB5) -> (no net)
- J5 pad B8: Net-(J5-PadB8) -> (no net)
- U2 pad 1: Net-(U2-Pad1) -> (no net)
- U2 pad 12: Net-(U2-Pad12) -> (no net)
- U2 pad 18: Net-(U2-Pad18) -> (no net)
- U2 pad 20: Net-(U2-Pad20) -> (no net)
- U2 pad 25: Net-(U2-Pad25) -> (no net)
- U2 pad 26: Net-(U2-Pad26) -> (no net)
- U2 pad 8: Net-(U2-Pad8) -> (no net)
- U3 pad 18: Net-(U3-Pad18) -> (no net)
- U3 pad 26: Net-(U3-Pad26) -> (no net)
