File: Hardware/0.3/Hub16.sch (KiCad schematic (older format))
At the start: 89 parts, among them J1 USB_C_Receptacle_USB2.0, J2 AVR-ISP-6, K1 KEYSW, K11 KEYSW, K12 KEYSW, K13 KEYSW, K14 KEYSW, K16 KEYSW, K17 KEYSW, K18 KEYSW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

Commit message: changing sw15/16 code
Parts:
- C1: Digikey PN (none) -> 1276-1871-1-ND; MPN (none) -> CL10A106MP8NNNC; Substitue Allowed? (none) -> Y
- C10, C11, C6, C7, C8, C9: Digikey PN (none) -> 1276-1000-1-ND; MPN (none) -> CL10B104KB8NNNC; Substitue Allowed? (none) -> Y
- C2, C3: Digikey PN (none) -> 1276-2228-1-ND; MPN (none) -> CL10C220JB8NFNC; Substitue Allowed? (none) -> Y
- C4, C5: Digikey PN (none) -> 1276-1866-1-ND; MPN (none) -> CL10A105MP8NNNC; Substitue Allowed? (none) -> Y
- D1: Digikey PN (none) -> 732-4980-1-ND; MPN (none) -> 150060VS75000; Substitue Allowed? (none) -> Y
- D10, D16, D2, D22, D23, D29, D3, D30, D31, D32, D4: Digikey PN (none) -> 1528-1104-ND; Substitue Allowed? (none) -> N
- D11, D12, D13, D14, D17, D18, D19, D20, D24, D25, D26, D27, D5, D6, D7, D8: Digikey PN (none) -> 1N4148W-FDICT-ND; Substitue Allowed? (none) -> Y
- F1: Digikey PN (none) -> 507-1813-1-ND; MPN FSMD050-0805-R -> 0ZCK0050FF2E; Notes (none) -> LCSC: Substitute PN; Substitue Allowed? (none) -> Y
- J1: Notes (none) -> Cannot source from Digikey, available on AliExpress: https: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; Substitue Allowed? (none) -> N
- JP11: DNP (none) -> DNP
- K1, K11, K12, K13, K14, K16, K17, K18, K19, K2, K3, K4, K6, K7, K8, K9: Notes Buy model without extra locating pins. (3 Pin) -> (none)
- R1: Digikey PN (none) -> CR0603-JW-222ELFCT-ND; MPN (none) -> CR0603-JW-222ELF; Substitue Allowed? (none) -> Y
- R11, R2, R5, R8: Digikey PN (none) -> CR0603-JW-103ELFCT-ND; MPN (none) -> CR0603-JW-103ELF; Substitue Allowed? (none) -> Y
- R3, R4: Digikey PN (none) -> 118-CR0603-JW-512ELFCT-ND; MPN (none) -> CR0603-JW-512ELF; Substitue Allowed? (none) -> Y
- R6, R7: Digikey PN (none) -> CR0603-JW-220ELFCT-ND; MPN (none) -> CR0603-JW-220ELF; Substitue Allowed? (none) -> Y
- RN1, RN3: Digikey PN (none) -> RAVF104DJT10K0CT-ND; MPN (none) -> RAVF104DJT10K0; Substitue Allowed? (none) -> Y
- SW1: Digikey PN (none) -> 401-1704-1-ND; MPN TSA343G00-250J2 -> KSR223GLFG; Notes (none) -> LCSC: Substitute PN; Substitue Allowed? (none) -> Y
- SW2, SW3: Digikey PN (none) -> 987-1398-ND; LCSC PN (none) -> C361165; MPN (none) -> EC11E1834403; Substitue Allowed? (none) -> Y
- U2: Digikey PN (none) -> ATMEGA32U4-AURCT-ND; Substitue Allowed? (none) -> N
- Y1: Digikey PN (none) -> 535-9134-1-ND; Substitue Allowed? (none) -> Y

Commit message: add images and start assembly instructions
Parts:
- RN1, RN3: symbol josh-passive:RN -> Hub16-rescue:RN-josh-passive
Changed lines of the file:
@@
 NoConn ~ 6650 3450
 $Comp
-L josh-passive:RN RN1
+L Hub16-rescue:RN-josh-passive RN1
 U 1 1 5DE76473
 P 4925 6875
@@
 $EndComp
 $Comp
-L josh-passive:RN RN1
+L Hub16-rescue:RN-josh-passive RN1
 U 2 1 5DE77B57
 P 5175 6575
@@
 $EndComp
 $Comp
-L josh-passive:RN RN1
+L Hub16-rescue:RN-josh-passive RN1
 U 3 1 5DE7C32C
 P 5475 6575
@@
 	5475 6350 5475 6375
 $Comp
-L josh-passive:RN RN3
+L Hub16-rescue:RN-josh-passive RN3
 U 2 1 5E2FAA67
 P 2025 6600
@@
 $EndComp
 $Comp
-L josh-passive:RN RN3
+L Hub16-rescue:RN-josh-passive RN3
 U 3 1 5E2FAA6D
 P 2325 6600
@@
 $EndComp
 $Comp
-L josh-passive:RN RN3
+L Hub16-rescue:RN-josh-passive RN3
 U 1 1 5E3B16E5
 P 1775 6900
@@
 	2400 850  2400 950
 $Comp
-L josh-passive:RN RN3
+L Hub16-rescue:RN-josh-passive RN3
 U 4 1 5DFFA8CC
 P 1775 7100
@@
 $EndComp
 $Comp
-L josh-passive:RN RN1
+L Hub16-rescue:RN-josh-passive RN1
 U 4 1 5E037CE5
 P 4925 7075

Commit message: r0.4 and hunting down bugs
Parts:
- C1: DigiKey (none) -> 1276-1871-1-ND; Digikey PN 1276-1871-1-ND -> (none); LCSC (none) -> C85713
- C10, C11, C6, C7, C8, C9: DigiKey (none) -> 1276-1000-1-ND; Digikey PN 1276-1000-1-ND -> (none); LCSC (none) -> C1591
- C2, C3: DigiKey (none) -> 1276-2228-1-ND; Digikey PN 1276-2228-1-ND -> (none); LCSC (none) -> C1653
- C4, C5: DigiKey (none) -> 1276-1866-1-ND; Digikey PN 1276-1866-1-ND -> (none); LCSC (none) -> C29936
- D1: DigiKey (none) -> 732-4980-1-ND; Digikey PN 732-4980-1-ND -> (none); LCSC (none) -> C364559
- D10, D16, D2, D22, D23, D29, D3, D30, D31, D32, D4: DigiKey (none) -> 1528-1104-ND; Digikey PN 1528-1104-ND -> (none); LCSC (none) -> WS2812B-B; LCSC PN WS2812B-B -> (none); Notes LCSC PN - Black Model -> LCSC - Black Model
- D11, D12, D13, D14, D17, D18, D19, D20, D24, D25, D26, D27, D5, D6, D7, D8: DigiKey (none) -> 1N4148W-FDICT-ND; Digikey PN 1N4148W-FDICT-ND -> (none); LCSC (none) -> C83528; LCSC PN C83528 -> (none)
- F1: DigiKey (none) -> 507-1813-1-ND; Digikey PN 507-1813-1-ND -> (none); LCSC (none) -> C181350; LCSC PN C181350 -> (none)
- J1: LCSC (none) -> C319148; LCSC PN C319148 -> (none)
- R1: DigiKey (none) -> CR0603-JW-222ELFCT-ND; Digikey PN CR0603-JW-222ELFCT-ND -> (none); LCSC (none) -> C113303
- R11, R2, R5, R8: DigiKey (none) -> CR0603-JW-103ELFCT-ND; Digikey PN CR0603-JW-103ELFCT-ND -> (none); LCSC (none) -> C144116
- R3, R4: DigiKey (none) -> 118-CR0603-JW-512ELFCT-ND; Digikey PN 118-CR0603-JW-512ELFCT-ND -> (none); LCSC (none) -> C14677
- R6, R7: DigiKey (none) -> CR0603-JW-220ELFCT-ND; Digikey PN CR0603-JW-220ELFCT-ND -> (none); LCSC (none) -> C203424
- RN1, RN3: DigiKey (none) -> RAVF104DJT10K0CT-ND; Digikey PN RAVF104DJT10K0CT-ND -> (none); LCSC (none) -> C136853
- SW1: DigiKey (none) -> 401-1704-1-ND; Digikey PN 401-1704-1-ND -> (none); LCSC (none) -> C354946; LCSC PN C354946 -> (none)
- SW2, SW3: DigiKey (none) -> 987-1398-ND; Digikey PN 987-1398-ND -> (none); LCSC (none) -> C361165; LCSC PN C361165 -> (none)
- U2: DigiKey (none) -> ATMEGA32U4-AURCT-ND; Digikey PN ATMEGA32U4-AURCT-ND -> (none); LCSC (none) -> C44854; LCSC PN C44854 -> (none)
- Y1: DigiKey (none) -> 535-9134-1-ND; Digikey PN 535-9134-1-ND -> (none); LCSC (none) -> C179641; LCSC PN C179641 -> (none)
