File: Hardware/0.4/usb-hub.sch (KiCad schematic (older format))
At the start: 27 parts, among them J3 USB_C_Receptacle_USB2.0, J4 USB_C_Receptacle_USB2.0, J5 USB_C_Receptacle_USB2.0, U1 TPD2S017, U3 CY7C65632-28LTXCT, Y2 12MHz

Commit message: r0.4 and hunting down bugs
Parts:
- removed R10: 100K, Resistor_SMD:R_0603_1608Metric, symbol Device:R
- removed U1: TPD2S017, Package_TO_SOT_SMD:SOT-23-6, symbol Power_Protection:TPD2S017
- added U1: USBLC6-2SC6, Package_TO_SOT_SMD:SOT-23-6, symbol josh-ic:USBLC6-2SC6
- C12, C13, C14, C15, C16, C17, C18, C19, C20, C21, C22: Manufacturer (none) -> Samsung Electro-Mechanics
- FB1, FB2, FB3, FB4: Manufacturer (none) -> Murata
- J3, J4, J5: footprint josh-connectors:USB_C_Receptacle_GT-USB-7010 -> josh-connectors:USB_C_U262-161N-4BVC11; Manufacturer (none) -> XKB Enterprise; Notes Cannot source from Digikey, available on AliExpress: https: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 -> Cannot source from DigiKey; Substitue Allowed? N -> Y
- R12, R13: Manufacturer (none) -> Bourns; Notes (none) -> LCSC: Substitute PN
- R14: Manufacturer (none) -> Rohm Semiconductor; Notes Cannot source from LCSC, no substitutes available -> Cannot source from LCSC
- R9: DNP DNP -> (none); Manufacturer (none) -> Bourns; Notes (none) -> LCSC: Substitute PN
- RN5: footprint Resistor_SMD:R_Array_Convex_4x0402 -> Resistor_SMD:R_Array_Convex_4x0603; Manufacturer (none) -> Bourns; Notes (none) -> LCSC: Substitute PN
- U3: footprint Package_DFN_QFN:QFN-28-1EP_5x5mm_P0.5mm_EP3.35x3.35mm_ThermalVias -> josh-dfn-qfn:QFN-28-1EP_5x5mm_P0.5mm_EP3.35x3.35mm_ThermalVias; Manufacturer (none) -> Cypress Semiconductor
- Y2: symbol Hub16-rescue:Crystal_GND24_Small-Device-Hub16-rescue -> Device:Crystal_GND24_Small; Manufacturer (none) -> Abracon LLC
Connections:
- net labels removed: GANG
- wire segments 174 -> 169
Other:
- note removed: "Figure out which\none to place"
- moved on the sheet: R14
