File: Hardware/0.5/Hub16.kicad_pcb (KiCad board)
At the start: 2 copper layers, 89 x 100 mm, 109 parts, among them J1 USB_C_Receptacle_USB2.0, J2 AVR-ISP-6, J3 USB_C_Receptacle_USB2.0, J4 USB_C_Receptacle_USB2.0, J5 USB_C_Receptacle_USB2.0, K1 KEYSW, K11 KEYSW, K12 KEYSW, K13 KEYSW, K14 KEYSW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

Commit message: updated documentation + wrote test script
Other:
- board text removed: "JLCJLC JLCJLC"
Changed lines of the file:
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@@
   (general
     (thickness 1.6)
-    (drawings 16)
+    (drawings 15)
     (tracks 1046)
     (zones 0)
@@
       (drillshape 0)
       (scaleselection 1)
-      (outputdirectory "gerbers/"))
+      (outputdirectory "assembly/"))
   )
   (net 0 "")
@@
       (effects (font (size 1 1) (thickness 0.15)) (justify mirror))
     )
-    (fp_text user 2020-03-30 (at -1.1 -1.3) (layer B.Mask)
-      (effects (font (size 1 1) (thickness 0.15)) (justify mirror))
+    (fp_text user Hub16 (at -1.7 2.4) (layer B.SilkS)
+      (effects (font (size 2 2) (thickness 0.2)) (justify mirror))
     )
     (fp_text user "Rev 0.5" (at -3.4 0.5) (layer B.SilkS)
       (effects (font (size 1 1) (thickness 0.15)) (justify mirror))
     )
-    (fp_text user Hub16 (at -1.7 2.4) (layer B.SilkS)
-      (effects (font (size 2 2) (thickness 0.2)) (justify mirror))
+    (fp_text user 2020-03-30 (at -1.1 -1.3) (layer B.Mask)
+      (effects (font (size 1 1) (thickness 0.15)) (justify mirror))
     )
   )
@@
     )
   )
-  (gr_text "JLCJLC\nJLCJLC" (at 92.5 77.5) (layer B.SilkS)
-    (effects (font (size 1 1) (thickness 0.15)) (justify mirror))
-  )
   (gr_text PROG (at 103.1 56.65) (layer B.SilkS)
     (effects (font (size 1 1) (thickness 0.15)) (justify mirror))
@@
   (segment (start 125.75 91.05) (end 123.9 91.05) (width 0.2) (layer B.Cu) (net 10))
   (segment (start 128.4 88.4) (end 125.75 91.05) (width 0.2) (layer B.Cu) (net 10))
-  (segment (start 127.9 100) (end 125.5 97.6) (width 0.2) (layer B.Cu) (net 11))
-  (segment (start 120.3 113.65) (end 120.55 113.65) (width 0.2) (layer B.Cu) (net 11))
+  (segment (start 127.9 107.6) (end 127.9 100) (width 0.2) (layer B.Cu) (net 11))
   (segment (start 125.45 110.05) (end 127.9 107.6) (width 0.2) (layer B.Cu) (net 11))
-  (segment (start 120.55 113.65) (end 124.15 110.05) (width 0.2) (layer B.Cu) (net 11))
   (segment (start 124.15 110.05) (end 125.45 110.05) (width 0.2) (layer B.Cu) (net 11))
+  (segment (start 120.3 113.65) (end 120.55 113.65) (width 0.2) (layer B.Cu) (net 11))
+  (segment (start 120.55 113.65) (end 124.15 110.05) (width 0.2) (layer B.Cu) (net 11))
+  (segment (start 127.9 100) (end 125.5 97.6) (width 0.2) (layer B.Cu) (net 11))
   (segment (start 125.5 97.6) (end 125.3 97.6) (width 0.2) (layer B.Cu) (net 11))
-  (segment (start 127.9 107.6) (end 127.9 100) (width 0.2) (layer B.Cu) (net 11))
   (segment (start 59.55 63.6) (end 59.55 66.64) (width 0.2) (layer B.Cu) (net 12))
   (segment (start 88.25 75.9) (end 86.9 75.9) (width 0.2) (layer B.Cu) (net 13))
@@
   (segment (start 88.5 132) (end 86.1 129.6) (width 0.2) (layer B.Cu) (net 30))
   (segment (start 86.1 129.6) (end 76.9 129.6) (width 0.2) (layer B.Cu) (net 30))
+  (segment (start 56.5 127.5) (end 56.5 122.5) (width 0.2) (layer B.Cu) (net 31))
+  (segment (start 57.94499 121.05501) (end 57.94499 121.05) (width 0.2) (layer B.Cu) (net 31))
+  (segment (start 56.5 122.5) (end 57.94499 121.05501) (width 0.2) (layer B.Cu) (net 31))
+  (segment (start 71.4 131.95) (end 60.95 131.95) (width 0.2) (layer B.Cu) (net 31))
   (segment (start 63.45 116.85) (end 63.7 116.85) (width 0.2) (layer B.Cu) (net 31))
-  (segment (start 61.19499 117.8) (end 62.5 117.8) (width 0.2) (layer B.Cu) (net 31))
   (segment (start 60.95 131.95) (end 56.5 127.5) (width 0.2) (layer B.Cu) (net 31))
   (segment (start 57.94499 121.05) (end 61.19499 117.8) (width 0.2) (layer B.Cu) (net 31))
-  (segment (start 71.4 131.95) (end 60.95 131.95) (width 0.2) (layer B.Cu) (net 31))
-  (segment (start 56.5 122.5) (end 57.94499 121.05501) (width 0.2) (layer B.Cu) (net 31))
+  (segment (start 61.19499 117.8) (end 62.5 117.8) (width 0.2) (layer B.Cu) (net 31))
   (segment (start 62.5 117.8) (end 63.45 116.85) (width 0.2) (layer B.Cu) (net 31))
-  (segment (start 57.94499 121.05501) (end 57.94499 121.05) (width 0.2) (layer B.Cu) (net 31))
-  (segment (start 56.5 127.5) (end 56.5 122.5) (width 0.2) (layer B.Cu) (net 31))
   (segment (start 116.7 64.25) (end 116.7 66.64) (width 0.2) (layer B.Cu) (net 32))
   (segment (start 116.7 83.45) (end 116.7 85.69) (width 0.2) (layer B.Cu) (net 33))
