File: Hardware/0.5/Hub16.sch (KiCad schematic (older format))
At the start: 83 parts, among them J1 USB_C_Receptacle_USB2.0, J2 AVR-ISP-6, K1 KEYSW, K11 KEYSW, K12 KEYSW, K13 KEYSW, K14 KEYSW, K16 KEYSW, K17 KEYSW, K18 KEYSW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

Commit message: correct RN part numbers + generate pdf of schematic
Parts:
- RN1, RN3: DigiKey RAVF104DJT10K0CT-ND -> RAVF164DJT10K0CT-ND; LCSC C136853 -> C107374; MPN RAVF104DJT10K0 -> RAVF164DJT10K0
Changed lines of the file:
@@
 F 2 "Resistor_SMD:R_Array_Convex_4x0603" V 4875 6850 50  0001 C CNN
 F 3 "~" V 4875 6850 50  0001 C CNN
-F 4 "RAVF104DJT10K0CT-ND" H 4875 6850 50  0001 C CNN "DigiKey"
-F 5 "RAVF104DJT10K0" H 4875 6850 50  0001 C CNN "MPN"
+F 4 "RAVF164DJT10K0CT-ND" H 4875 6850 50  0001 C CNN "DigiKey"
+F 5 "RAVF164DJT10K0" H 4875 6850 50  0001 C CNN "MPN"
 F 6 "Y" H 4875 6850 50  0001 C CNN "Substitue Allowed?"
-F 7 "C136853" H 4875 6850 50  0001 C CNN "LCSC"
+F 7 "C107374" H 4875 6850 50  0001 C CNN "LCSC"
 F 8 "Bourns" H 4875 6850 50  0001 C CNN "Manufacturer"
 F 9 "LCSC: Substitute PN" H 4875 6850 50  0001 C CNN "Notes"
@@
 F 2 "Resistor_SMD:R_Array_Convex_4x0603" V 5125 6550 50  0001 C CNN
 F 3 "~" V 5125 6550 50  0001 C CNN
-F 4 "RAVF104DJT10K0CT-ND" H 5125 6550 50  0001 C CNN "DigiKey"
-F 5 "RAVF104DJT10K0" H 5125 6550 50  0001 C CNN "MPN"
+F 4 "RAVF164DJT10K0CT-ND" H 5125 6550 50  0001 C CNN "DigiKey"
+F 5 "RAVF164DJT10K0" H 5125 6550 50  0001 C CNN "MPN"
 F 6 "Y" H 5125 6550 50  0001 C CNN "Substitue Allowed?"
-F 7 "C136853" H 5125 6550 50  0001 C CNN "LCSC"
+F 7 "C107374" H 5125 6550 50  0001 C CNN "LCSC"
 F 8 "Bourns" H 5125 6550 50  0001 C CNN "Manufacturer"
 F 9 "LCSC: Substitute PN" H 5125 6550 50  0001 C CNN "Notes"
@@
 F 2 "Resistor_SMD:R_Array_Convex_4x0603" V 5425 6550 50  0001 C CNN
 F 3 "~" V 5425 6550 50  0001 C CNN
-F 4 "RAVF104DJT10K0CT-ND" H 5425 6550 50  0001 C CNN "DigiKey"
-F 5 "RAVF104DJT10K0" H 5425 6550 50  0001 C CNN "MPN"
+F 4 "RAVF164DJT10K0CT-ND" H 5425 6550 50  0001 C CNN "DigiKey"
+F 5 "RAVF164DJT10K0" H 5425 6550 50  0001 C CNN "MPN"
 F 6 "Y" H 5425 6550 50  0001 C CNN "Substitue Allowed?"
-F 7 "C136853" H 5425 6550 50  0001 C CNN "LCSC"
+F 7 "C107374" H 5425 6550 50  0001 C CNN "LCSC"
 F 8 "Bourns" H 5425 6550 50  0001 C CNN "Manufacturer"
 F 9 "LCSC: Substitute PN" H 5425 6550 50  0001 C CNN "Notes"
@@
 F 2 "Resistor_SMD:R_Array_Convex_4x0603" V 1975 6575 50  0001 C CNN
 F 3 "~" V 1975 6575 50  0001 C CNN
-F 4 "RAVF104DJT10K0CT-ND" H 1975 6575 50  0001 C CNN "DigiKey"
-F 5 "RAVF104DJT10K0" H 1975 6575 50  0001 C CNN "MPN"
+F 4 "RAVF164DJT10K0CT-ND" H 1975 6575 50  0001 C CNN "DigiKey"
+F 5 "RAVF164DJT10K0" H 1975 6575 50  0001 C CNN "MPN"
 F 6 "Y" H 1975 6575 50  0001 C CNN "Substitue Allowed?"
-F 7 "C136853" H 1975 6575 50  0001 C CNN "LCSC"
+F 7 "C107374" H 1975 6575 50  0001 C CNN "LCSC"
 F 8 "Bourns" H 1975 6575 50  0001 C CNN "Manufacturer"
 F 9 "LCSC: Substitute PN" H 1975 6575 50  0001 C CNN "Notes"
@@
 F 2 "Resistor_SMD:R_Array_Convex_4x0603" V 2275 6575 50  0001 C CNN
 F 3 "~" V 2275 6575 50  0001 C CNN
-F 4 "RAVF104DJT10K0CT-ND" H 2275 6575 50  0001 C CNN "DigiKey"
-F 5 "RAVF104DJT10K0" H 2275 6575 50  0001 C CNN "MPN"
+F 4 "RAVF164DJT10K0CT-ND" H 2275 6575 50  0001 C CNN "DigiKey"
+F 5 "RAVF164DJT10K0" H 2275 6575 50  0001 C CNN "MPN"
 F 6 "Y" H 2275 6575 50  0001 C CNN "Substitue Allowed?"
-F 7 "C136853" H 2275 6575 50  0001 C CNN "LCSC"
+F 7 "C107374" H 2275 6575 50  0001 C CNN "LCSC"
 F 8 "Bourns" H 2275 6575 50  0001 C CNN "Manufacturer"
 F 9 "LCSC: Substitute PN" H 2275 6575 50  0001 C CNN "Notes"
@@
 F 2 "Resistor_SMD:R_Array_Convex_4x0603" V 1725 6875 50  0001 C CNN
 F 3 "~" V 1725 6875 50  0001 C CNN
-F 4 "RAVF104DJT10K0CT-ND" H 1725 6875 50  0001 C CNN "DigiKey"
-F 5 "RAVF104DJT10K0" H 1725 6875 50  0001 C CNN "MPN"
+F 4 "RAVF164DJT10K0CT-ND" H 1725 6875 50  0001 C CNN "DigiKey"
+F 5 "RAVF164DJT10K0" H 1725 6875 50  0001 C CNN "MPN"
 F 6 "Y" H 1725 6875 50  0001 C CNN "Substitue Allowed?"
-F 7 "C136853" H 1725 6875 50  0001 C CNN "LCSC"
+F 7 "C107374" H 1725 6875 50  0001 C CNN "LCSC"
 F 8 "Bourns" H 1725 6875 50  0001 C CNN "Manufacturer"
 F 9 "LCSC: Substitute PN" H 1725 6875 50  0001 C CNN "Notes"
@@
 F 2 "Resistor_SMD:R_Array_Convex_4x0603" V 1725 7075 50  0001 C CNN
 F 3 "~" V 1725 7075 50  0001 C CNN
-F 4 "RAVF104DJT10K0CT-ND" H 1725 7075 50  0001 C CNN "DigiKey"
-F 5 "RAVF104DJT10K0" H 1725 7075 50  0001 C CNN "MPN"
+F 4 "RAVF164DJT10K0CT-ND" H 1725 7075 50  0001 C CNN "DigiKey"
+F 5 "RAVF164DJT10K0" H 1725 7075 50  0001 C CNN "MPN"
 F 6 "Y" H 1725 7075 50  0001 C CNN "Substitue Allowed?"
-F 7 "C136853" H 1725 7075 50  0001 C CNN "LCSC"
+F 7 "C107374" H 1725 7075 50  0001 C CNN "LCSC"
 F 8 "Bourns" H 1725 7075 50  0001 C CNN "Manufacturer"
 F 9 "LCSC: Substitute PN" H 1725 7075 50  0001 C CNN "Notes"
@@
 F 2 "Resistor_SMD:R_Array_Convex_4x0603" V 4875 7050 50  0001 C CNN
 F 3 "~" V 4875 7050 50  0001 C CNN
-F 4 "RAVF104DJT10K0CT-ND" H 4875 7050 50  0001 C CNN "DigiKey"
-F 5 "RAVF104DJT10K0" H 4875 7050 50  0001 C CNN "MPN"
+F 4 "RAVF164DJT10K0CT-ND" H 4875 7050 50  0001 C CNN "DigiKey"
+F 5 "RAVF164DJT10K0" H 4875 7050 50  0001 C CNN "MPN"
 F 6 "Y" H 4875 7050 50  0001 C CNN "Substitue Allowed?"
-F 7 "C136853" H 4875 7050 50  0001 C CNN "LCSC"
+F 7 "C107374" H 4875 7050 50  0001 C CNN "LCSC"
 F 8 "Bourns" H 4875 7050 50  0001 C CNN "Manufacturer"
 F 9 "LCSC: Substitute PN" H 4875 7050 50  0001 C CNN "Notes"

Commit message: fix v0.5 bom + release prototypes
Parts:
- RN1, RN3: LCSC C107374 -> C29718
Changed lines of the file:
@@
 F 5 "RAVF164DJT10K0" H 4875 6850 50  0001 C CNN "MPN"
 F 6 "Y" H 4875 6850 50  0001 C CNN "Substitue Allowed?"
-F 7 "C107374" H 4875 6850 50  0001 C CNN "LCSC"
+F 7 "C29718" H 4875 6850 50  0001 C CNN "LCSC"
 F 8 "Bourns" H 4875 6850 50  0001 C CNN "Manufacturer"
 F 9 "LCSC: Substitute PN" H 4875 6850 50  0001 C CNN "Notes"
@@
 F 5 "RAVF164DJT10K0" H 5125 6550 50  0001 C CNN "MPN"
 F 6 "Y" H 5125 6550 50  0001 C CNN "Substitue Allowed?"
-F 7 "C107374" H 5125 6550 50  0001 C CNN "LCSC"
+F 7 "C29718" H 5125 6550 50  0001 C CNN "LCSC"
 F 8 "Bourns" H 5125 6550 50  0001 C CNN "Manufacturer"
 F 9 "LCSC: Substitute PN" H 5125 6550 50  0001 C CNN "Notes"
@@
 F 5 "RAVF164DJT10K0" H 5425 6550 50  0001 C CNN "MPN"
 F 6 "Y" H 5425 6550 50  0001 C CNN "Substitue Allowed?"
-F 7 "C107374" H 5425 6550 50  0001 C CNN "LCSC"
+F 7 "C29718" H 5425 6550 50  0001 C CNN "LCSC"
 F 8 "Bourns" H 5425 6550 50  0001 C CNN "Manufacturer"
 F 9 "LCSC: Substitute PN" H 5425 6550 50  0001 C CNN "Notes"
@@
 F 5 "RAVF164DJT10K0" H 1975 6575 50  0001 C CNN "MPN"
 F 6 "Y" H 1975 6575 50  0001 C CNN "Substitue Allowed?"
-F 7 "C107374" H 1975 6575 50  0001 C CNN "LCSC"
+F 7 "C29718" H 1975 6575 50  0001 C CNN "LCSC"
 F 8 "Bourns" H 1975 6575 50  0001 C CNN "Manufacturer"
 F 9 "LCSC: Substitute PN" H 1975 6575 50  0001 C CNN "Notes"
@@
 F 5 "RAVF164DJT10K0" H 2275 6575 50  0001 C CNN "MPN"
 F 6 "Y" H 2275 6575 50  0001 C CNN "Substitue Allowed?"
-F 7 "C107374" H 2275 6575 50  0001 C CNN "LCSC"
+F 7 "C29718" H 2275 6575 50  0001 C CNN "LCSC"
 F 8 "Bourns" H 2275 6575 50  0001 C CNN "Manufacturer"
 F 9 "LCSC: Substitute PN" H 2275 6575 50  0001 C CNN "Notes"
@@
 F 5 "RAVF164DJT10K0" H 1725 6875 50  0001 C CNN "MPN"
 F 6 "Y" H 1725 6875 50  0001 C CNN "Substitue Allowed?"
-F 7 "C107374" H 1725 6875 50  0001 C CNN "LCSC"
+F 7 "C29718" H 1725 6875 50  0001 C CNN "LCSC"
 F 8 "Bourns" H 1725 6875 50  0001 C CNN "Manufacturer"
 F 9 "LCSC: Substitute PN" H 1725 6875 50  0001 C CNN "Notes"
@@
 F 5 "RAVF164DJT10K0" H 1725 7075 50  0001 C CNN "MPN"
 F 6 "Y" H 1725 7075 50  0001 C CNN "Substitue Allowed?"
-F 7 "C107374" H 1725 7075 50  0001 C CNN "LCSC"
+F 7 "C29718" H 1725 7075 50  0001 C CNN "LCSC"
 F 8 "Bourns" H 1725 7075 50  0001 C CNN "Manufacturer"
 F 9 "LCSC: Substitute PN" H 1725 7075 50  0001 C CNN "Notes"
@@
 F 5 "RAVF164DJT10K0" H 4875 7050 50  0001 C CNN "MPN"
 F 6 "Y" H 4875 7050 50  0001 C CNN "Substitue Allowed?"
-F 7 "C107374" H 4875 7050 50  0001 C CNN "LCSC"
+F 7 "C29718" H 4875 7050 50  0001 C CNN "LCSC"
 F 8 "Bourns" H 4875 7050 50  0001 C CNN "Manufacturer"
 F 9 "LCSC: Substitute PN" H 4875 7050 50  0001 C CNN "Notes"
