File: Hardware/0.5/usb-hub.sch (KiCad schematic (older format))
At the start: 26 parts, among them J3 USB_C_Receptacle_USB2.0, J4 USB_C_Receptacle_USB2.0, J5 USB_C_Receptacle_USB2.0, U1 USBLC6-2SC6, U3 CY7C65632-28LTXCT, Y2 12MHz

Commit message: correct RN part numbers + generate pdf of schematic
Parts:
- RN5: DigiKey RAVF104DJT10K0CT-ND -> RAVF164DJT10K0CT-ND; LCSC C136853 -> C107374; MPN RAVF104DJT10K0 -> RAVF164DJT10K0
Changed lines of the file:
@@
 F 2 "Resistor_SMD:R_Array_Convex_4x0603" V 6350 7050 50  0001 C CNN
 F 3 "~" H 6075 7050 50  0001 C CNN
-F 4 "RAVF104DJT10K0CT-ND" H 6075 7050 50  0001 C CNN "DigiKey"
-F 5 "RAVF104DJT10K0" H 6075 7050 50  0001 C CNN "MPN"
+F 4 "RAVF164DJT10K0CT-ND" H 6075 7050 50  0001 C CNN "DigiKey"
+F 5 "RAVF164DJT10K0" H 6075 7050 50  0001 C CNN "MPN"
 F 6 "Y" H 6075 7050 50  0001 C CNN "Substitue Allowed?"
-F 7 "C136853" H 6075 7050 50  0001 C CNN "LCSC"
+F 7 "C107374" H 6075 7050 50  0001 C CNN "LCSC"
 F 8 "Bourns" H 6075 7050 50  0001 C CNN "Manufacturer"
 F 9 "LCSC: Substitute PN" H 6075 7050 50  0001 C CNN "Notes"

Commit message: fix v0.5 bom + release prototypes
Parts:
- RN5: LCSC C107374 -> C29718
Changed lines of the file:
@@
 F 5 "RAVF164DJT10K0" H 6075 7050 50  0001 C CNN "MPN"
 F 6 "Y" H 6075 7050 50  0001 C CNN "Substitue Allowed?"
-F 7 "C107374" H 6075 7050 50  0001 C CNN "LCSC"
+F 7 "C29718" H 6075 7050 50  0001 C CNN "LCSC"
 F 8 "Bourns" H 6075 7050 50  0001 C CNN "Manufacturer"
 F 9 "LCSC: Substitute PN" H 6075 7050 50  0001 C CNN "Notes"
