File: Hardware/0.6/usb-hub.sch (KiCad schematic (older format))
At the start: 37 parts, among them J3 USB_C_Receptacle_USB2.0, J4 USB_C_Receptacle_USB2.0, J5 USB_C_Receptacle_USB2.0, U1 USBLC6-2SC6, U3 CY7C65632-28LTXCT, U4 USBLC6-2SC6, U5 USBLC6-2SC6, U6 USBLC6-2SC6, Y2 12MHz

Commit message: more layout
Connections:
- net D1_D+: now also U5.4 (IO2); no longer U5.1 (IO1)
- net D1_D-: now also U5.6 (IO1); no longer U5.3 (IO2)
- net D2_D+: now also U6.4 (IO2); no longer U6.3 (IO2)
- net D2_D-: now also U6.6 (IO1); no longer U6.1 (IO1)
- net D3_D+: now also U4.4 (IO2); no longer U4.3 (IO2)
- net D3_D-: now also U4.6 (IO1); no longer U4.1 (IO1)
- net at J4.A6 (D+), J4.B6 (D+): now also U5.3 (IO2); no longer U5.6 (IO1)
- net at J4.A7 (D-), J4.B7 (D-): now also U5.1 (IO1); no longer U5.4 (IO2)
- net at J3.A6 (D+), J3.B6 (D+): now also U6.3 (IO2); no longer U6.4 (IO2)
- net at J3.A7 (D-), J3.B7 (D-): now also U6.1 (IO1); no longer U6.6 (IO1)
- net at J5.A6 (D+), J5.B6 (D+): now also U4.3 (IO2); no longer U4.4 (IO2)
- net at J5.A7 (D-), J5.B7 (D-): now also U4.1 (IO1); no longer U4.6 (IO1)
Changed lines of the file:
@@
 Downstream Ports
 Wire Wire Line
-	6525 1950 6175 1950
-Wire Wire Line
-	6175 1750 6525 1750
+	6525 1750 6175 1750
+Wire Wire Line
+	6175 1950 6525 1950
+Text Label 6175 1950 0    50   ~ 0
+D1_D+
 Text Label 6175 1750 0    50   ~ 0
-D1_D+
-Text Label 6175 1950 0    50   ~ 0
 D1_D-
 NoConn ~ 7925 1400
@@
 F 7 "STmicroelectronics" H 8925 4025 50  0001 C CNN "Manufacturer"
 	1    8925 4025
-	1    0    0    -1
+	-1   0    0    -1
 $EndComp
 Wire Wire Line
@@
 F 7 "STmicroelectronics" H 6525 5250 50  0001 C CNN "Manufacturer"
 	1    6525 5250
-	1    0    0    -1
+	-1   0    0    -1
 $EndComp
 Wire Wire Line
@@
 	3000 2625 3000 3200
 Wire Wire Line
-	7900 1900 7900 1950
-Wire Wire Line
-	7900 1700 7900 1750
-Wire Wire Line
-	7900 1750 7650 1750
-Wire Wire Line
-	7650 1750 7650 1950
-Connection ~ 7900 1750
-Wire Wire Line
-	7900 1750 7900 1800
-Wire Wire Line
 	6925 2300 6925 2400
 $Comp
@@
 F 7 "STmicroelectronics" H 6925 1850 50  0001 C CNN "Manufacturer"
 	1    6925 1850
-	1    0    0    -1
-$EndComp
-Wire Wire Line
-	7325 1950 7650 1950
-Wire Wire Line
-	7325 1750 7550 1750
-Wire Wire Line
-	7550 1750 7550 1875
-Wire Wire Line
-	7550 1875 7800 1875
-Wire Wire Line
-	7800 1875 7800 1950
-Wire Wire Line
-	7800 1950 7900 1950
+	-1   0    0    -1
+$EndComp
+Wire Wire Line
+	7900 1700 7900 1750
+Wire Wire Line
+	7900 1900 7900 1950
+Wire Wire Line
+	7325 1950 7900 1950
 Connection ~ 7900 1950
 Wire Wire Line
 	7900 1950 7900 2000
+Wire Wire Line
+	7325 1750 7900 1750
+Connection ~ 7900 1750
+Wire Wire Line
+	7900 1750 7900 1800
 $EndSCHEMATC

Commit message: update gitignore
Parts:
- removed C23: 1u, Capacitor_SMD:C_0603_1608Metric, symbol Device:C
- removed R13: 100K, Resistor_SMD:R_0603_1608Metric, symbol Device:R
- C12: value 100n -> 10u
- C13: value 10u -> 100n
- F2, F3, F4: value 500mA -> 200mA
- R10: value 47K -> 10K; DigiKey CR0603-JW-103ELFCT-ND -> (none); LCSC C144116 -> (none); MPN CR0603-JW-103ELF -> (none); Manufacturer Bourns -> (none); Notes LCSC: Substitute PN -> (none); Substitue Allowed? Y -> (none)
- R12: DigiKey CR0603-JW-103ELFCT-ND -> (none); LCSC C144116 -> (none); MPN CR0603-JW-103ELF -> (none); Manufacturer Bourns -> (none); Notes LCSC: Substitute PN -> (none); Substitue Allowed? Y -> (none)
- R9: value 100K -> 10K
Connections:
- net +3V3: now also R10.2, R12.2
- net +5V: no longer R12.1
- net GND: no longer R10.2
- net at R10.1, U3.17 (nRESET): no longer R12.2
- net at U3.22 (SELF_PWR): now also R12.1
Changed lines of the file:
@@
 P 1300 7050
 F 0 "C12" H 1415 7096 50  0000 L CNN
-F 1 "100n" H 1415 7005 50  0000 L CNN
+F 1 "10u" H 1415 7005 50  0000 L CNN
 F 2 "Capacitor_SMD:C_0603_1608Metric" H 1338 6900 50  0001 C CNN
 F 3 "~" H 1300 7050 50  0001 C CNN
@@
 P 1850 7050
 F 0 "C13" H 1965 7096 50  0000 L CNN
-F 1 "10u" H 1965 7005 50  0000 L CNN
+F 1 "100n" H 1965 7005 50  0000 L CNN
 F 2 "Capacitor_SMD:C_0603_1608Metric" H 1888 6900 50  0001 C CNN
 F 3 "~" H 1850 7050 50  0001 C CNN
@@
 NoConn ~ 4025 2375
 NoConn ~ 4025 2475
-$Comp
-L Device:R R12
-U 1 1 5E7EC2E6
-P 2525 3025
-F 0 "R12" H 2650 3075 50  0000 C CNN
-F 1 "10K" H 2650 3000 50  0000 C CNN
-F 2 "Resistor_SMD:R_0603_1608Metric" V 2455 3025 50  0001 C CNN
-F 3 "~" H 2525 3025 50  0001 C CNN
-F 4 "CR0603-JW-103ELFCT-ND  " H 2525 3025 50  0001 C CNN "DigiKey"
-F 5 "CR0603-JW-103ELF " H 2525 3025 50  0001 C CNN "MPN"
-F 6 "Y" H 2525 3025 50  0001 C CNN "Substitue Allowed?"
-F 7 "C144116" H 2525 3025 50  0001 C CNN "LCSC"
-F 8 "Bourns" H 2525 3025 50  0001 C CNN "Manufacturer"
-F 9 "LCSC: Substitute PN" H 2525 3025 50  0001 C CNN "Notes"
-	1    2525 3025
-	1    0    0    -1
-$EndComp
 $Comp
 L Device:C C?
@@
 Wire Wire Line
 	2150 2175 2700 2175
-$Comp
-L Device:R R9
-U 1 1 5E6ABC35
-P 3550 3100
-F 0 "R9" H 3650 3150 50  0000 C CNN
-F 1 "100K" H 3700 3075 50  0000 C CNN
-F 2 "Resistor_SMD:R_0603_1608Metric" V 3480 3100 50  0001 C CNN
-F 3 "~" H 3550 3100 50  0001 C CNN
-F 4 "" H 3675 3025 50  0001 C CNN "DNP"
-F 5 "CR0603-JW-104ELFCT-ND " H 3550 3100 50  0001 C CNN "DigiKey"
-F 6 "CR0603-JW-104ELF " H 3550 3100 50  0001 C CNN "MPN"
-F 7 "Y" H 3550 3100 50  0001 C CNN "Substitue Allowed?"
-F 8 "C203223" H 3550 3100 50  0001 C CNN "LCSC"
-F 9 "Bourns" H 3550 3100 50  0001 C CNN "Manufacturer"
-F 10 "LCSC: Substitute PN" H 3550 3100 50  0001 C CNN "Notes"
-	1    3550 3100
-	1    0    0    -1
-$EndComp
 Wire Wire Line
 	3550 3325 3550 3250
@@
 P 6700 1200
 F 0 "F3" V 6475 1200 50  0000 C CNN
-F 1 "500mA" V 6566 1200 50  0000 C CNN
+F 1 "200mA" V 6566 1200 50  0000 C CNN
 F 2 "josh-passives-smt:Fuse_0805_2012Metric" H 6750 1000 50  0001 L CNN
 F 3 "~" H 6700 1200 50  0001 C CNN
@@
 P 8700 3375
 F 0 "F4" V 8475 3375 50  0000 C CNN
-F 1 "500mA" V 8566 3375 50  0000 C CNN
+F 1 "200mA" V 8566 3375 50  0000 C CNN
 F 2 "josh-passives-smt:Fuse_0805_2012Metric" H 8750 3175 50  0001 L CNN
 F 3 "~" H 8700 3375 50  0001 C CNN
@@
 P 6300 4600
 F 0 "F2" V 6075 4600 50  0000 C CNN
-F 1 "500mA" V 6166 4600 50  0000 C CNN
+F 1 "200mA" V 6166 4600 50  0000 C CNN
 F 2 "josh-passives-smt:Fuse_0805_2012Metric" H 6350 4400 50  0001 L CNN
 F 3 "~" H 6300 4600 50  0001 C CNN
@@
 Wire Wire Line
 	6525 4600 7350 4600
-$Comp
-L Device:R R13
-U 1 1 5F3E2D7A
-P 3225 3100
-F 0 "R13" H 3350 3150 50  0000 C CNN
-F 1 "100K" H 3375 3075 50  0000 C CNN
-F 2 "Resistor_SMD:R_0603_1608Metric" V 3155 3100 50  0001 C CNN
-F 3 "~" H 3225 3100 50  0001 C CNN
-F 4 "" H 3350 3025 50  0001 C CNN "DNP"
-F 5 "CR0603-JW-104ELFCT-ND " H 3225 3100 50  0001 C CNN "DigiKey"
-F 6 "CR0603-JW-104ELF " H 3225 3100 50  0001 C CNN "MPN"
-F 7 "Y" H 3225 3100 50  0001 C CNN "Substitue Allowed?"
-F 8 "C203223" H 3225 3100 50  0001 C CNN "LCSC"
-F 9 "Bourns" H 3225 3100 50  0001 C CNN "Manufacturer"
-F 10 "LCSC: Substitute PN" H 3225 3100 50  0001 C CNN "Notes"
-	1    3225 3100
-	1    0    0    -1
-$EndComp
-Wire Wire Line
-	3225 3325 3225 3250
-$Comp
-L power:GND #PWR010
-U 1 1 5F3E2D81
-P 3225 3325
-F 0 "#PWR010" H 3225 3075 50  0001 C CNN
-F 1 "GND" H 3230 3152 50  0000 C CNN
-F 2 "" H 3225 3325 50  0001 C CNN
-F 3 "" H 3225 3325 50  0001 C CNN
-	1    3225 3325
-	1    0    0    -1
-$EndComp
-Wire Wire Line
-	3225 2725 4025 2725
-Wire Wire Line
-	3225 2725 3225 2950
-$Comp
-L Device:R R10
-U 1 1 5F417231
-P 2525 3425
-F 0 "R10" H 2650 3475 50  0000 C CNN
-F 1 "47K" H 2650 3400 50  0000 C CNN
-F 2 "Resistor_SMD:R_0603_1608Metric" V 2455 3425 50  0001 C CNN
-F 3 "~" H 2525 3425 50  0001 C CNN
-F 4 "CR0603-JW-103ELFCT-ND  " H 2525 3425 50  0001 C CNN "DigiKey"
-F 5 "CR0603-JW-103ELF " H 2525 3425 50  0001 C CNN "MPN"
-F 6 "Y" H 2525 3425 50  0001 C CNN "Substitue Allowed?"
-F 7 "C144116" H 2525 3425 50  0001 C CNN "LCSC"
-F 8 "Bourns" H 2525 3425 50  0001 C CNN "Manufacturer"
-F 9 "LCSC: Substitute PN" H 2525 3425 50  0001 C CNN "Notes"
-	1    2525 3425
-	1    0    0    -1
-$EndComp
-$Comp
-L Device:C C23
-U 1 1 5F417E16
-P 2200 3425
-F 0 "C23" H 2315 3471 50  0000 L CNN
-F 1 "1u" H 2315 3380 50  0000 L CNN
-F 2 "Capacitor_SMD:C_0603_1608Metric" H 2238 3275 50  0001 C CNN
-F 3 "~" H 2200 3425 50  0001 C CNN
-	1    2200 3425
-	1    0    0    -1
-$EndComp
-Wire Wire Line
-	2525 3275 2525 3250
-Wire Wire Line
-	2200 3250 2525 3250
-Connection ~ 2525 3250
-Wire Wire Line
-	2525 3250 2525 3200
-Wire Wire Line
-	2525 3200 3000 3200
-Wire Wire Line
-	3000 2625 4025 2625
-Connection ~ 2525 3200
-Wire Wire Line
-	2525 3200 2525 3175
-Wire Wire Line
-	2200 3250 2200 3275
-Wire Wire Line
-	2525 3650 2525 3575
-$Comp
-L power:GND #PWR09
-U 1 1 5F469822
-P 2525 3650
-F 0 "#PWR09" H 2525 3400 50  0001 C CNN
-F 1 "GND" H 2530 3477 50  0000 C CNN
-F 2 "" H 2525 3650 50  0001 C CNN
-F 3 "" H 2525 3650 50  0001 C CNN
-	1    2525 3650
-	1    0    0    -1
-$EndComp
-Wire Wire Line
-	2200 3650 2200 3575
-$Comp
-L power:GND #PWR06
-U 1 1 5F473DDC
-P 2200 3650
-F 0 "#PWR06" H 2200 3400 50  0001 C CNN
-F 1 "GND" H 2205 3477 50  0000 C CNN
-F 2 "" H 2200 3650 50  0001 C CNN
-F 3 "" H 2200 3650 50  0001 C CNN
-	1    2200 3650
-	1    0    0    -1
-$EndComp
-$Comp
-L power:+5V #PWR?
-U 1 1 5F47FCDA
-P 2525 2850
-AR Path="/5F47FCDA" Ref="#PWR?"  Part="1"
-AR Path="/5E5406D9/5F47FCDA" Ref="#PWR08"  Part="1"
-F 0 "#PWR08" H 2525 2700 50  0001 C CNN
-F 1 "+5V" H 2525 3000 50  0000 C CNN
-F 2 "" H 2525 2850 50  0001 C CNN
-F 3 "" H 2525 2850 50  0001 C CNN
-	1    2525 2850
-	1    0    0    -1
-$EndComp
-Wire Wire Line
-	2525 2850 2525 2875
-Wire Wire Line
-	3000 2625 3000 3200
 Wire Wire Line
 	6925 2300 6925 2400
@@
 Wire Wire Line
 	7900 1750 7900 1800
+$Comp
+L Device:R R12
+U 1 1 5F35A109
+P 3825 2725
+F 0 "R12" V 3775 2525 50  0000 C CNN
+F 1 "10K" V 3825 2725 50  0000 C CNN
+F 2 "Resistor_SMD:R_0603_1608Metric" V 3755 2725 50  0001 C CNN
+F 3 "~" H 3825 2725 50  0001 C CNN
+	1    3825 2725
+	0    1    1    0
+$EndComp
+$Comp
+L Device:R R10
+U 1 1 5F35B149
+P 3825 2625
+F 0 "R10" V 3775 2425 50  0000 C CNN
+F 1 "10K" V 3825 2625 50  0000 C CNN
+F 2 "Resistor_SMD:R_0603_1608Metric" V 3755 2625 50  0001 C CNN
+F 3 "~" H 3825 2625 50  0001 C CNN
+	1    3825 2625
+	0    1    1    0
+$EndComp
+Wire Wire Line
+	3975 2625 4025 2625
+Wire Wire Line
+	4025 2725 3975 2725
+Wire Wire Line
+	3675 2725 3550 2725
+Wire Wire Line
+	3550 2725 3550 2625
+Wire Wire Line
+	3675 2625 3550 2625
+Connection ~ 3550 2625
+Wire Wire Line
+	3550 2625 3550 2575
+$Comp
+L power:+3.3V #PWR06
+U 1 1 5F38B684
+P 3550 2575
+F 0 "#PWR06" H 3550 2425 50  0001 C CNN
+F 1 "+3.3V" H 3565 2748 50  0000 C CNN
+F 2 "" H 3550 2575 50  0001 C CNN
+F 3 "" H 3550 2575 50  0001 C CNN
+	1    3550 2575
+	1    0    0    -1
+$EndComp
+$Comp
+L Device:R R9
+U 1 1 5E6ABC35
+P 3550 3100
+F 0 "R9" H 3650 3150 50  0000 C CNN
+F 1 "10K" H 3675 3075 50  0000 C CNN
+F 2 "Resistor_SMD:R_0603_1608Metric" V 3480 3100 50  0001 C CNN
+F 3 "~" H 3550 3100 50  0001 C CNN
+F 4 "" H 3675 3025 50  0001 C CNN "DNP"
+F 5 "CR0603-JW-104ELFCT-ND " H 3550 3100 50  0001 C CNN "DigiKey"
+F 6 "CR0603-JW-104ELF " H 3550 3100 50  0001 C CNN "MPN"
+F 7 "Y" H 3550 3100 50  0001 C CNN "Substitue Allowed?"
+F 8 "C203223" H 3550 3100 50  0001 C CNN "LCSC"
+F 9 "Bourns" H 3550 3100 50  0001 C CNN "Manufacturer"
+F 10 "LCSC: Substitute PN" H 3550 3100 50  0001 C CNN "Notes"
+	1    3550 3100
+	1    0    0    -1
+$EndComp
 $EndSCHEMATC
