File: Hardware/0.6/Hub16.kicad_pcb (KiCad board)
At the start: 2 copper layers, 89 x 100 mm, 119 parts, among them J1 USB_C_Receptacle_USB2.0, J2 AVR-ISP-6, J3 USB_C_Receptacle_USB2.0, J4 USB_C_Receptacle_USB2.0, J5 USB_C_Receptacle_USB2.0, K1 KEYSW, K11 KEYSW, K12 KEYSW, K13 KEYSW, K14 KEYSW, K16 KEYSW, K17 KEYSW, K18 KEYSW, K19 KEYSW, K2 KEYSW, K3 KEYSW, K4 KEYSW, K6 KEYSW, K7 KEYSW, K8 KEYSW, K9 KEYSW, SW1 KMR2, SW2 Rotary_Encoder_Switch, SW3 Rotary_Encoder_Switch, U1 USBLC6-2SC6, U2 ATMEGA32U4, U3 CY7C65632-28LTXCT, U4 USBLC6-2SC6, U5 USBLC6-2SC6, U6 USBLC6-2SC6, Y1 16MHz, Y2 12MHz

Commit message: robustness ++
Parts:
- added C23: 100n, Capacitor_SMD:C_0603_1608Metric, B.Cu at (94.5, 85.1)
- added C27: 100n, Capacitor_SMD:C_0603_1608Metric, B.Cu at (84.1, 73.5)
- added C28: 100n, Capacitor_SMD:C_0603_1608Metric, B.Cu at (59.6, 80.6)
- added C29: 100n, Capacitor_SMD:C_0603_1608Metric, B.Cu at (55.8, 60.4)
- added C30: 100n, Capacitor_SMD:C_0603_1608Metric, B.Cu at (59.6, 99.8)
- added C31: 100n, Capacitor_SMD:C_0603_1608Metric, B.Cu at (76.6, 131.2)
- added C32: 100n, Capacitor_SMD:C_0603_1608Metric, B.Cu at (125.2, 110.9)
- added C33: 100n, Capacitor_SMD:C_0603_1608Metric, B.Cu at (59.5, 118.8)
- added C34: 100n, Capacitor_SMD:C_0603_1608Metric, B.Cu at (95.6, 131.2)
- added C35: 100n, Capacitor_SMD:C_0603_1608Metric, B.Cu at (128.1, 53.2)
- added C36: 100n, Capacitor_SMD:C_0603_1608Metric, B.Cu at (125.2, 91.6)
- added C37: 100n, Capacitor_SMD:C_0603_1608Metric, B.Cu at (114.7, 131.2)
- added C38: 100n, Capacitor_SMD:C_0603_1608Metric, B.Cu at (125.2, 72.6)
Connections:
- net Net-(D22-Pad2) renamed /LED_1
Routing:
- net +5V: track 15.9 -> 38.0 mm, vias 5 -> 3
- net GND: track 89.4 -> 99.6 mm, vias 70 -> 83
- net /SCK: track 20.3 -> 17.8 mm, vias 0 -> 2
- net /MOSI: track 17.1 -> 15.2 mm
- net /row2: track 66.8 -> 66.7 mm, vias 0 -> 2
