File: Hardware/0.6/Hub16.sch (KiCad schematic (older format))
At the start: 83 parts, among them J1 USB_C_Receptacle_USB2.0, J2 AVR-ISP-6, K1 KEYSW, K11 KEYSW, K12 KEYSW, K13 KEYSW, K14 KEYSW, K16 KEYSW, K17 KEYSW, K18 KEYSW, K19 KEYSW, K2 KEYSW, K3 KEYSW, K4 KEYSW, K6 KEYSW, K7 KEYSW, K8 KEYSW, K9 KEYSW, SW1 KMR2, SW2 Rotary_Encoder_Switch, SW3 Rotary_Encoder_Switch, U2 ATMEGA32U4, Y1 16MHz

Commit message: update gitignore
Parts:
- R1: value 2K2 -> 5K1
Changed lines of the file:
@@
 P 9800 5050
 F 0 "R1" H 9870 5096 50  0000 L CNN
-F 1 "2K2" H 9870 5005 50  0000 L CNN
+F 1 "5K1" H 9870 5005 50  0000 L CNN
 F 2 "Resistor_SMD:R_0603_1608Metric" V 9730 5050 50  0001 C CNN
 F 3 "~" H 9800 5050 50  0001 C CNN

Commit message: laid out USB hub from scratch, much better
Parts:
- added FB5: 600R, josh-passives-smt:Ferrite_Bead_0603, symbol josh-passive:Ferrite_Bead_PWR
Connections:
- net +5V: now also U2.2 (UVcc), U2.7 (VBus), FB5.1; no longer F1.1
- net VBUS: no longer U2.2 (UVcc), U2.7 (VBus)
- new net: F1.1, FB5.2
Changed lines of the file:
@@
-	1    0    0    -1
-$EndComp
-$Comp
-L power:VBUS #PWR016
-U 1 1 5CC6529C
-P 4700 2025
-F 0 "#PWR016" H 4700 1875 50  0001 C CNN
-F 1 "VBUS" H 4700 2175 50  0000 C CNN
-F 2 "" H 4700 2025 50  0001 C CNN
-F 3 "" H 4700 2025 50  0001 C CNN
-	1    4700 2025
 	1    0    0    -1
 $EndComp
@@
 $EndComp
 Wire Wire Line
-	2800 1225 2850 1225
-Wire Wire Line
-	2850 1225 2850 1175
+	3175 1225 3225 1225
+Wire Wire Line
+	3225 1225 3225 1175
 $Comp
 L power:+5V #PWR0111
 U 1 1 5EB49DE7
-P 2850 1175
+P 3225 1175
 AR Path="/5EB49DE7" Ref="#PWR0111"  Part="1"
 AR Path="/5E5406D9/5EB49DE7" Ref="#PWR?"  Part="1"
-F 0 "#PWR0111" H 2850 1025 50  0001 C CNN
-F 1 "+5V" H 2850 1325 50  0000 C CNN
-F 2 "" H 2850 1175 50  0001 C CNN
-F 3 "" H 2850 1175 50  0001 C CNN
-	1    2850 1175
+F 0 "#PWR0111" H 3225 1025 50  0001 C CNN
+F 1 "+5V" H 3225 1325 50  0000 C CNN
+F 2 "" H 3225 1175 50  0001 C CNN
+F 3 "" H 3225 1175 50  0001 C CNN
+	1    3225 1175
 	1    0    0    -1
 $EndComp
@@
 	1    0    0    -1
 $EndComp
-Connection ~ 2850 1225
+Connection ~ 3225 1225
 $Comp
 L Connector:USB_C_Receptacle_USB2.0 J?
@@
 	1825 1975 1825 1925
 Wire Wire Line
-	3025 1225 3025 1200
-Wire Wire Line
-	2850 1225 3025 1225
+	3400 1225 3400 1200
+Wire Wire Line
+	3225 1225 3400 1225
 Text Label 2500 1775 2    50   ~ 0
 USB_UP_D-
@@
 L power:PWR_FLAG #FLG0101
 U 1 1 5EB49E07
-P 3025 1200
+P 3400 1200
 AR Path="/5EB49E07" Ref="#FLG0101"  Part="1"
 AR Path="/5E5406D9/5EB49E07" Ref="#FLG?"  Part="1"
-F 0 "#FLG0101" H 3025 1275 50  0001 C CNN
-F 1 "PWR_FLAG" V 3025 1328 50  0000 L CNN
-F 2 "" H 3025 1200 50  0001 C CNN
-F 3 "~" H 3025 1200 50  0001 C CNN
-	1    3025 1200
+F 0 "#FLG0101" H 3400 1275 50  0001 C CNN
+F 1 "PWR_FLAG" V 3400 1328 50  0000 L CNN
+F 2 "" H 3400 1200 50  0001 C CNN
+F 3 "~" H 3400 1200 50  0001 C CNN
+	1    3400 1200
 	1    0    0    -1
 $EndComp
@@
 Wire Wire Line
 	8750 5075 8950 5075
+$Comp
+L josh-passive:Ferrite_Bead_PWR FB5
+U 1 1 5F3B3001
+P 3025 1225
+AR Path="/5F3B3001" Ref="FB5"  Part="1"
+AR Path="/5E5406D9/5F3B3001" Ref="FB?"  Part="1"
+F 0 "FB5" H 3025 1075 50  0000 C CNN
+F 1 "600R" H 3025 1400 50  0000 C CNN
+F 2 "josh-passives-smt:Ferrite_Bead_0603" H 3025 1155 50  0001 C CNN
+F 3 "~" V 3025 1225 50  0001 C CNN
+F 4 "C19330" H 3025 1225 50  0001 C CNN "LCSC"
+F 5 "BLM18AG601SN1D" H 3025 1225 50  0001 C CNN "MPN"
+F 6 "490-1014-1-ND" H 3025 1225 50  0001 C CNN "DigiKey"
+F 7 "Y" H 3025 1225 50  0001 C CNN "Substitue Allowed?"
+F 8 "Murata" H 3025 1225 50  0001 C CNN "Manufacturer"
+	1    3025 1225
+	1    0    0    1
+$EndComp
+Wire Wire Line
+	2875 1225 2800 1225
+$Comp
+L power:+5V #PWR?
+U 1 1 5F4541D8
+P 4700 2000
+F 0 "#PWR?" H 4700 1850 50  0001 C CNN
+F 1 "+5V" H 4715 2173 50  0000 C CNN
+F 2 "" H 4700 2000 50  0001 C CNN
+F 3 "" H 4700 2000 50  0001 C CNN
+	1    4700 2000
+	-1   0    0    -1
+$EndComp
+Wire Wire Line
+	4700 2000 4700 2025
 $EndSCHEMATC

Commit message: robustness ++
Parts:
- added C23, C27, C28, C29, C30, C31, C32, C33, C34, C35, C36, C37, C38: 100n, Capacitor_SMD:C_0603_1608Metric, symbol Device:C
Connections:
- net +5V: now also FB5.2, C23.1, C27.1, C28.1, C29.1, C30.1, C31.1, C32.1, C33.1, C34.1, C35.1, C36.1, C37.1, C38.2; no longer FB5.1
- net GND: now also C23.2, C27.2, C28.2, C29.2, C30.2, C31.2, C32.2, C33.2, C34.2, C35.2, C36.2, C37.2, C38.1
- net LED_1: now reaches D22.2 (DOUT), D23.4 (DIN)
- net at F1.1: now also FB5.1; no longer FB5.2
Other:
- moved on the sheet: C10, C11, C5, C6, C7, C8, C9, D1, D10, D16, D2, D22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
