File: Production/1.0-hs-test-fixture/Hub16.kicad_pcb (KiCad board)
At the start: 2 copper layers, 89 x 100 mm, 84 parts, among them J1 USB_C_Receptacle_USB2.0, J2 AVR-ISP-6, J3 AVR-ISP-6, J4 AVR-ISP-6, J5 Conn_01x02_Male, K1 Kailh Hotswap Socket, K11 Kailh Hotswap Socket, K12 Kailh Hotswap Socket, K13 Kailh Hotswap Socket, K14 Kailh Hotswap Socket, K16 Kailh Hotswap Socket, K17 Kailh Hotswap Socket, K18 Kailh Hotswap Socket, K19 Kailh Hotswap Socket, K2 Kailh Hotswap Socket, K3 Kailh Hotswap Socket, K4 Kailh Hotswap Socket, K6 Kailh Hotswap Socket, K7 Kailh Hotswap Socket, K8 Kailh Hotswap Socket, K9 Kailh Hotswap Socket, Q1 BSS138, Q10 BSS138, Q11 BSS138, Q12 BSS138, Q13 BSS138, Q14 BSS138, Q15 BSS138, Q16 BSS138, Q2 BSS138, Q3 BSS138, Q4 BSS138, Q5 BSS138, Q6 BSS138, Q7 BSS138, Q8 BSS138, Q9 BSS138, SW1 EVQPUL, SW2 EC11 Encoder, SW3 EC11 Encoder, U1 74HC595, U2 ATMEGA32U4, U3 74HC595, Y1 16MHz

Commit message: update bare-bones spelling + text fixture update
Parts:
- removed R8: 5K1, Resistor_SMD:R_0603_1608Metric
Connections:
- RN2 pad 1: (no net) -> /MCU_T_nRST
- RN2 pad 8: (no net) -> /T_nRST
Routing:
- net /T_nRST: track 49.2 -> 73.4 mm, vias 0 -> 2
- net /MCU_T_nRST: track 34.7 -> 16.9 mm
